Commit message: RGBD camera

File: ros_ws/src/turtlebot3_simulations/turtlebot3_gazebo/urdf/turtlebot3_burger.urdf (robot description, URDF)
Before this commit: robot turtlebot3_burger, 7 links, 6 joints
Links:
- removed link base_scan
- added link camera_link; collision box size=0.015 0.030 0.027
- added link camera_rgb_frame
- added link camera_rgb_optical_frame
Joints:
- removed joint scan_joint
- added joint camera_joint: type fixed, parent base_link, child camera_link, origin xyz=0.040 -0.000 0.110 rpy=0 0 0
- added joint camera_rgb_joint: type fixed, parent camera_link, child camera_rgb_frame, origin xyz=0.003 0.000 0.009 rpy=0 0 0
- added joint camera_rgb_optical_joint: type fixed, parent camera_rgb_frame, child camera_rgb_optical_frame, origin xyz=0 0 0 rpy=-1.5707 0 -1.57
